File: flight controller.kicad_sch (KiCad schematic)
At the start: 71 parts, among them J1 Receiver, J10 Conn_01x03_Pin, J11 Conn_01x03_Pin, J12 Input Power, J13 Video In, J14 Video Out, J15 UART2, J16 I2C2, J17 UART3, J18 Analog, J2 SWD, J3 LED Strip, J4 Conn_01x03_Pin, J5 Conn_01x03_Pin, J6 Conn_01x03_Pin, J7 Conn_01x03_Pin, J8 Conn_01x03_Pin, J9 Conn_01x03_Pin, U1 STM32H743VITx, U2 AP2114HA-3.3TRG1, U3 AT7456E, U4 ICM-42688-P, U5 BMP388, U6 LIS3MDLTR, Y1 32.768kHz, Y2 16MHz, Y3 Crystal

Commit message: finished pcb
Parts:
- removed C10, C11, C12: 100nF, symbol Device:C
- removed C20, C28, C29: 1uF, symbol Device:C
- removed Card1: TF PUSH, lcsc:TF-SMD_TF-PUSH, symbol lcsc:TFPUSH
- removed J1: Receiver, symbol Connector:Conn_01x04_Pin
- removed J14: Video Out, symbol Connector:Conn_01x03_Pin
- removed J17: UART3, symbol Connector:Conn_01x06_Pin
- removed J18: Analog, symbol Connector:Conn_01x08_Pin
- removed USB1: TYPE-C 16PIN 2MD(073), lcsc:USB-C-SMD_TYPE-C-6PIN-2MD-073, symbol lcsc:TYPE-C16PIN2MD(073)
- added C13, C9: 100nF, Capacitor_SMD:C_0805_2012Metric, symbol Device:C
- added C3: 1uF, Capacitor_SMD:C_0805_2012Metric, symbol Device:C
- added D1, D2, D3, D4: WS2812B, LED_SMD:LED_WS2812B_PLCC4_5.0x5.0mm_P3.2mm, symbol LED:WS2812B
- added D5: 1N4001, Diode_THT:D_DO-41_SOD81_P7.62mm_Horizontal, symbol Device:D
- added D6: LED, LED_SMD:LED_0805_2012Metric, symbol Device:LED
- added J12: M11, Connector_JST:JST_XH_B3B-XH-A_1x03_P2.50mm_Vertical, symbol Connector:Conn_01x03_Pin
- added J13: M12, Connector_JST:JST_XH_B3B-XH-A_1x03_P2.50mm_Vertical, symbol Connector:Conn_01x03_Pin
- added J16: Video Out, Connector_JST:JST_XH_B3B-XH-A_1x03_P2.50mm_Vertical, symbol Connector:Conn_01x03_Pin
- added J19: UART7, Connector_JST:JST_XH_B6B-XH-A_1x06_P2.50mm_Vertical, symbol Connector:Conn_01x06_Pin
- added J21: UART5, Connector_JST:JST_XH_B4B-XH-A_1x04_P2.50mm_Vertical, symbol Connector:Conn_01x04_Pin
- added J22: UART8, Connector_JST:JST_XH_B4B-XH-A_1x04_P2.50mm_Vertical, symbol Connector:Conn_01x04_Pin
- added J23: UART3, Connector_JST:JST_XH_B4B-XH-A_1x04_P2.50mm_Vertical, symbol Connector:Conn_01x04_Pin
- added J24: UART4, Connector_JST:JST_XH_B4B-XH-A_1x04_P2.50mm_Vertical, symbol Connector:Conn_01x04_Pin
- added J25: USB_C_Receptacle_USB2.0_16P, Connector_USB:USB_C_Receptacle_HCTL_HC-TYPE-C-16P-01A, symbol Connector:USB_C_Receptacle_USB2.0_16P
- added J26: Micro_SD_Card, lcsc:TF-SMD_TF-PUSH, symbol Connector:Micro_SD_Card
- added J27: GPIO, Connector_JST:JST_XH_B10B-XH-A_1x10_P2.50mm_Vertical, symbol Connector:Conn_01x10_Pin
- added J3: M2, Connector_JST:JST_XH_B3B-XH-A_1x03_P2.50mm_Vertical, symbol Connector:Conn_01x03_Pin
- added J4: M3, Connector_JST:JST_XH_B3B-XH-A_1x03_P2.50mm_Vertical, symbol Connector:Conn_01x03_Pin
- added R1, R10, R3, R5, R7, R9: 10K, Resistor_SMD:R_0805_2012Metric, symbol Device:R
- added R19: 56, Resistor_SMD:R_0805_2012Metric, symbol Device:R
- C1, C2, C27: footprint (none) -> Capacitor_SMD:C_0805_2012Metric
- C10: renamed from C26; footprint (none) -> Capacitor_SMD:C_0805_2012Metric
- C11: renamed from C25; footprint (none) -> Capacitor_SMD:C_0805_2012Metric
- C12: renamed from C7; footprint (none) -> Capacitor_THT:CP_Radial_D8.0mm_P3.50mm
- C14: renamed from C19; footprint (none) -> Capacitor_SMD:C_0805_2012Metric
- C15: renamed from C18; footprint (none) -> Capacitor_SMD:C_0805_2012Metric
- C16: renamed from C30; footprint (none) -> Capacitor_SMD:C_0805_2012Metric
- C17: renamed from C24; footprint (none) -> Capacitor_SMD:C_0805_2012Metric
- C18: renamed from C22; footprint (none) -> Capacitor_THT:CP_Radial_D8.0mm_P3.50mm
- C19: renamed from C21; footprint (none) -> Capacitor_SMD:C_0805_2012Metric
- C20: renamed from C23; footprint (none) -> Capacitor_SMD:C_0805_2012Metric
- C21: renamed from C3; footprint (none) -> Capacitor_SMD:C_0805_2012Metric
- C22: renamed from C4; footprint (none) -> Capacitor_SMD:C_0805_2012Metric
- C23: renamed from C8; footprint (none) -> Capacitor_SMD:C_0805_2012Metric
- C24: renamed from C5; footprint (none) -> Capacitor_SMD:C_0805_2012Metric
- C25: renamed from C9; footprint (none) -> Capacitor_SMD:C_0805_2012Metric
- C26: renamed from C6; footprint (none) -> Capacitor_SMD:C_0805_2012Metric
- C4: renamed from C15; footprint (none) -> Capacitor_SMD:C_0805_2012Metric
- C5: renamed from C14; footprint (none) -> Capacitor_SMD:C_0805_2012Metric
- C6: renamed from C13; footprint (none) -> Capacitor_SMD:C_0805_2012Metric
- C7: renamed from C17; footprint (none) -> Capacitor_SMD:C_0805_2012Metric
- C8: renamed from C16; footprint (none) -> Capacitor_SMD:C_0805_2012Metric
- J1: renamed from J12; footprint (none) -> Connector_AMASS:AMASS_XT30PW-M_1x02_P2.50mm_Horizontal
- J10: value Conn_01x03_Pin -> M9; footprint (none) -> Connector_JST:JST_XH_B3B-XH-A_1x03_P2.50mm_Vertical
- J11: value Conn_01x03_Pin -> M10; footprint (none) -> Connector_JST:JST_XH_B3B-XH-A_1x03_P2.50mm_Vertical
- J14: renamed from J13; footprint (none) -> Connector_JST:JST_XH_B3B-XH-A_1x03_P2.50mm_Vertical
- J15: renamed from J3; footprint (none) -> Connector_JST:JST_XH_B3B-XH-A_1x03_P2.50mm_Vertical
- J17: renamed from J16; value I2C2 -> I2C4; footprint (none) -> Connector_JST:JST_XH_B4B-XH-A_1x04_P2.50mm_Vertical
- J18: renamed from J15; footprint (none) -> Connector_JST:JST_XH_B6B-XH-A_1x06_P2.50mm_Vertical
- J2: renamed from J4; value Conn_01x03_Pin -> M1; footprint (none) -> Connector_JST:JST_XH_B3B-XH-A_1x03_P2.50mm_Vertical
- J20: renamed from J2; footprint (none) -> Connector_JST:JST_XH_B6B-XH-A_1x06_P2.50mm_Vertical
- J5: value Conn_01x03_Pin -> M4; footprint (none) -> Connector_JST:JST_XH_B3B-XH-A_1x03_P2.50mm_Vertical
- J6: value Conn_01x03_Pin -> M5; footprint (none) -> Connector_JST:JST_XH_B3B-XH-A_1x03_P2.50mm_Vertical
- J7: value Conn_01x03_Pin -> M6; footprint (none) -> Connector_JST:JST_XH_B3B-XH-A_1x03_P2.50mm_Vertical
- J8: value Conn_01x03_Pin -> M7; footprint (none) -> Connector_JST:JST_XH_B3B-XH-A_1x03_P2.50mm_Vertical
- J9: value Conn_01x03_Pin -> M8; footprint (none) -> Connector_JST:JST_XH_B3B-XH-A_1x03_P2.50mm_Vertical
- R11: renamed from R2; footprint (none) -> Resistor_SMD:R_0805_2012Metric
- R12: value R -> 5.6K; footprint (none) -> Resistor_SMD:R_0805_2012Metric
- R13: value R -> 10K; footprint (none) -> Resistor_SMD:R_0805_2012Metric
- R14: renamed from R1; footprint (none) -> Resistor_SMD:R_0805_2012Metric
- R15: renamed from R8; footprint (none) -> Resistor_SMD:R_0805_2012Metric
- R16: renamed from R7; footprint (none) -> Resistor_SMD:R_0805_2012Metric
- R17: renamed from R3; footprint (none) -> Resistor_SMD:R_0805_2012Metric
- R18: renamed from R4; footprint (none) -> Resistor_SMD:R_0805_2012Metric
- R2: renamed from R9; footprint (none) -> Resistor_SMD:R_0805_2012Metric
- R4: renamed from R10; footprint (none) -> Resistor_SMD:R_0805_2012Metric
- R6: renamed from R5; footprint (none) -> Resistor_SMD:R_0805_2012Metric
- R8: renamed from R6; footprint (none) -> Resistor_SMD:R_0805_2012Metric
- U1: renamed from U2; footprint lcsc:SOT-223-3_L6.5-W3.4-P2.30-LS7.0-BR -> Package_TO_SOT_SMD:SOT-223
- U2: renamed from U5; footprint lcsc:SENSORM-SMD_BMP388 -> Package_LGA:ST_HLGA-10_2x2mm_P0.5mm_LayoutBorder3x2y
- U3: renamed from U6; footprint lcsc:LGA-12_L2.0-W2.0-P0.50-BL -> Package_LGA:LGA-12_2x2mm_P0.5mm
- U5: renamed from U3; footprint lcsc:TSSOP-28_L9.7-W4.4-P0.65-LS6.4-BL-EP-2 -> Package_SO:TSSOP-28-1EP_4.4x9.7mm_P0.65mm_EP2.85x6.7mm
- U6: renamed from U4; footprint lcsc:LGA-14_L3.0-W2.5-P0.50-TL -> Package_LGA:LGA-14_3x2.5mm_P0.5mm_LayoutBorder3x4y
- Y1: renamed from Y3; value Crystal -> 27MHz; footprint (none) -> Crystal:Crystal_HC49-U_Vertical
- Y2: footprint (none) -> Crystal:Crystal_HC49-U_Vertical
- Y3: renamed from Y1; footprint (none) -> Crystal:Crystal_DS26_D2.0mm_L6.0mm_Horizontal
- renumbered U1 to U4
Connections:
- net +3.3V: now also C27.2, C5.2, C8.2, J20.5 (Pin_5), R2.1, R4.1, C13.2, C3.2, C9.2, J26.4 (VDD), R1.2, R10.2, R3.2, R5.2, R7.2, R9.2; no longer C27.1, C5.1, C8.1, J17.2 (Pin_2), J20.2 (Pin_2), R2.2, R4.2
- net +5V: now also J15.2 (Pin_2), J17.3 (Pin_3), J18.5 (Pin_5), D5.2 (A), J12.2 (Pin_2), J13.2 (Pin_2), J16.2 (Pin_2), J19.5 (Pin_5), J21.3 (Pin_3), J22.3 (Pin_3), J23.3 (Pin_3), J24.3 (Pin_3), J27.1 (Pin_1), J3.2 (Pin_2), J4.2 (Pin_2); no longer J15.3 (Pin_3), J18.2 (Pin_2)
- net A1: now also U4.28 (PA4), J27.2 (Pin_2); no longer U4.30 (PA6)
- net A2: now also U4.29 (PA5), J27.3 (Pin_3); no longer U4.31 (PA7)
- net A3: now also U4.30 (PA6), J27.4 (Pin_4); no longer U4.32 (PC4)
- net A4: now also U4.31 (PA7), J27.5 (Pin_5); no longer U4.33 (PC5)
- net A5: now also U4.32 (PC4), J27.6 (Pin_6); no longer U4.34 (PB0)
- net A6: now also U4.33 (PC5), J27.7 (Pin_7); no longer U4.35 (PB1)
- net BOOT0: now also J20.4 (Pin_4); no longer J20.6 (Pin_6)
- net GND: now also C21.2, C23.2, C24.2, C25.2, C27.1, C5.1, C8.1, J10.3 (Pin_3), J11.3 (Pin_3), J14.3 (Pin_3), J15.3 (Pin_3), J17.4 (Pin_4), J18.6 (Pin_6), J2.3 (Pin_3), J20.6 (Pin_6), J5.3 (Pin_3), J6.3 (Pin_3), J7.3 (Pin_3), J8.3 (Pin_3), J9.3 (Pin_3), R11.2, R14.2, U5.29 (EP), C13.1, C3.1, C9.1, D1.3 (VSS), D2.3 (VSS), D3.3 (VSS), D4.3 (VSS), J12.3 (Pin_3), J13.3 (Pin_3), J16.3 (Pin_3), J19.6 (Pin_6), J21.4 (Pin_4), J22.4 (Pin_4), J23.4 (Pin_4), J24.4 (Pin_4), J25.A1 (GND), J25.A12 (GND), J25.B1 (GND), J25.B12 (GND), J25.S1 (SHIELD), J26.6 (VSS), J26.9 (SHIELD), J27.10 (Pin_10), J3.3 (Pin_3), J4.3 (Pin_3), R19.2; no longer C21.1, C23.1, C24.1, C25.1, C27.2, C5.2, C8.2, J10.1 (Pin_1), J11.1 (Pin_1), J14.1 (Pin_1), J15.1 (Pin_1), J17.1 (Pin_1), J18.1 (Pin_1), J2.1 (Pin_1), J20.1 (Pin_1), J5.1 (Pin_1), J6.1 (Pin_1), J7.1 (Pin_1), J8.1 (Pin_1), J9.1 (Pin_1), R11.1, R14.1
- net LED: now also U4.67 (PA8), D1.4 (DIN); no longer J15.2 (Pin_2)
- net M1: now also J2.1 (Pin_1), U4.43 (PE13); no longer J2.3 (Pin_3)
- net M2: now also U4.44 (PE14), J3.1 (Pin_1); no longer J5.3 (Pin_3)
- net M3: now also U4.46 (PB10), J4.1 (Pin_1); no longer J6.3 (Pin_3)
- net M4: now also J5.1 (Pin_1), U4.47 (PB11); no longer J7.3 (Pin_3)
- net M5: now also J6.1 (Pin_1), U4.61 (PD14); no longer J8.3 (Pin_3)
- net M6: now also J7.1 (Pin_1), U4.62 (PD15); no longer J9.3 (Pin_3)
- net M7: now also J8.1 (Pin_1), U4.63 (PC6); no longer J10.3 (Pin_3)
- net M8: now also J9.1 (Pin_1), U4.64 (PC7); no longer J11.3 (Pin_3)
- net NRST: now also J20.3 (Pin_3); no longer J20.5 (Pin_5)
- net OSC_32_IN: now also C24.1; no longer C24.2
- net OSC_IN: now also C21.1; no longer C21.2
- net SD_CK: now also J26.5 (CLK), R10.1
- net SD_CMD: now also J26.3 (CMD), R1.1
- net SD_D0: now also J26.7 (DAT0), R3.1
- net SD_D1: now also J26.8 (DAT1), R5.1
- net SD_D2: now also J26.1 (DAT2), R7.1
- net SD_D3: now also J26.2 (DAT3/CD), R9.1
- net SWCLK: now also J20.2 (Pin_2); no longer J20.4 (Pin_4)
- net SWDIO: now also J20.1 (Pin_1); no longer J20.3 (Pin_3)
- net UART2_CTS: now also J18.3 (Pin_3); no longer J18.5 (Pin_5)
- net UART2_RTS: now also J18.4 (Pin_4); no longer J18.6 (Pin_6)
- net UART2_RX: now also J18.2 (Pin_2); no longer J18.4 (Pin_4)
- net UART2_TX: now also J18.1 (Pin_1); no longer J18.3 (Pin_3)
- net UART3_RX: now also J23.2 (Pin_2)
- net UART3_TX: now also J23.1 (Pin_1)
- net USB_DN: now also U4.70 (PA11), J25.A7 (D-), J25.B7 (D-)
- net USB_DP: now also U4.71 (PA12), J25.A6 (D+), J25.B6 (D+)
- net VBUS: now also R12.1, J25.A4 (VBUS), J25.A9 (VBUS), J25.B4 (VBUS), J25.B9 (VBUS); no longer R12.2
- net VBUS_SENSE: now also R12.2, U4.68 (PA9); no longer R12.1
- net VCAP: now also C23.1, C25.1; no longer C23.2, C25.2
- net VIDEO_IN: now also J14.1 (Pin_1); no longer J14.3 (Pin_3)
- net VIDEO_OUT: now also R15.1, J16.1 (Pin_1); no longer R15.2
- net at C18.2: now also R15.2; no longer R15.1
- net ARM_LED: now reaches U4.2 (PE3)
- net ARM_LED: now also D6.2 (A)
- net UART7_RX: now reaches U4.37 (PE7)
- net UART7_RX: now also J19.2 (Pin_2)
- net UART7_TX: now reaches U4.38 (PE8)
- net UART7_TX: now also J19.1 (Pin_1)
- net UART7_RTS: now reaches U4.39 (PE9)
- net UART7_RTS: now also J19.4 (Pin_4)
- net UART7_CTS: now reaches U4.40 (PE10)
- net UART7_CTS: now also J19.3 (Pin_3)
- net UART5_RX: now reaches U4.51 (PB12)
- net UART5_RX: now also J21.2 (Pin_2)
- net UART5_TX: now reaches U4.52 (PB13)
- net UART5_TX: now also J21.1 (Pin_1)
- net M9: now reaches U4.60 (PD13)
- net M9: now also J10.1 (Pin_1)
- net UART4_RX: now reaches U4.81 (PD0)
- net UART4_RX: now also J24.2 (Pin_2)
- net UART4_TX: now reaches U4.82 (PD1)
- net UART4_TX: now also J24.1 (Pin_1)
- net I2C4_SCL: now reaches U4.95 (PB8)
- net I2C4_SCL: now also J17.1 (Pin_1), R2.2
- net I2C4_SDA: now reaches U4.96 (PB9)
- net I2C4_SDA: now also J17.2 (Pin_2), R4.2
- net UART8_RX: now reaches U4.97 (PE0)
- net UART8_RX: now also J22.2 (Pin_2)
- net UART8_TX: now reaches U4.98 (PE1)
- net UART8_TX: now also J22.1 (Pin_1)
- removed net I2C2_SCL: J17.4 (Pin_4), R2.1, U4.46 (PB10)
- removed net I2C2_SDA: J17.3 (Pin_3), R4.1, U4.47 (PB11)
- net RECEIVER_RX renamed M11
- net M11: now also J12.1 (Pin_1)
- net RECEIVER_TX renamed M12
- net M12: now also J13.1 (Pin_1)
- net UART3_CTS: no longer names the net of U4.58 (PD11)
- net UART3_RTS renamed M10
- net M10: now also J11.1 (Pin_1)
- new net: D6.1 (K), R19.1
- new net: D1.1 (VDD), D2.1 (VDD), D3.1 (VDD), D4.1 (VDD), D5.1 (K)
- new net: D4.2 (DOUT), J15.1 (Pin_1)
- new net: D3.2 (DOUT), D4.4 (DIN)
- new net: D2.2 (DOUT), D3.4 (DIN)
- new net: D1.2 (DOUT), D2.4 (DIN)
- new net: J25.B5 (CC2), R14.1
- new net: J25.A5 (CC1), R11.1
- new net A7: J27.8 (Pin_8), U4.34 (PB0)
- new net A8: J27.9 (Pin_9), U4.35 (PB1)
- no-connect marks 21 -> 20
Other:
- moved on the sheet: C10, C11, C12, C14, C15, C16, C17, C18, C19, C20, C21, C22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
