File: hardware/flight controller.kicad_pcb (KiCad board)
At the start: 4 copper layers, 50.2 x 98.1 mm, 92 parts, among them J1 Input Power, J10 M9, J11 M10, J12 M11, J13 M12, J14 Video In, J15 LED Strip, J16 Video Out, J17 I2C4, J18 UART2, J19 UART7, J2 M1, J20 SWD, J21 UART5, J22 UART8, J23 UART3, J24 UART4, J25 USB_C_Receptacle_USB2.0_16P, J26 Micro_SD_Card, J27 GPIO, J3 M2, J4 M3, J5 M4, J6 M5, J7 M6, J8 M7, J9 M8, U1 AP2114HA-3.3TRG1, U2 BMP388, U3 LIS3MDLTR, U4 STM32H743VITx, U5 AT7456E, U6 ICM-42688-P, Y1 27MHz, Y2 16MHz, Y3 32.768kHz

Commit message: finished bom
Parts:
- removed the C14 at (143.5, 111.5)
- removed the C15 at (145.5, 111.5)
- added C16: 100nF, Capacitor_SMD:C_0805_2012Metric, F.Cu at (145.0, 111.5)
- added C17: 4.7uF, Capacitor_SMD:C_0805_2012Metric, F.Cu at (143.0, 111.5)
- added C3: 47pF, Capacitor_SMD:C_0805_2012Metric, F.Cu at (138.0, 153.5)
- added C4: 22uF, Capacitor_SMD:C_1206_3216Metric, F.Cu at (137.0, 144.0)
- added C5: 22uF, Capacitor_SMD:C_1206_3216Metric, F.Cu at (137.0, 146.5)
- added L1: 6.8uH, Inductor_SMD:L_APV_APH0630, F.Cu at (143.0, 151.0)
- added R2: 100K, Resistor_SMD:R_0805_2012Metric, F.Cu at (136.0, 153.5)
- added R8: 22K, Resistor_SMD:R_0805_2012Metric, F.Cu at (136.0, 150.0)
- C1: value 4.7uF -> 100nF
- C2: value 4.7uF -> 10uF
- R10: renamed from R8; value 4.7K -> 3.3K
- R19: value 56 -> 75
- R3: renamed from R2; value 4.7K -> 3.3K
- R5: renamed from R4; value 4.7K -> 3.3K
- R7: renamed from R6; value 4.7K -> 3.3K
- U1: value AP2114HA-3.3TRG1 -> TPS54302; footprint Package_TO_SOT_SMD:SOT-223 -> Package_TO_SOT_SMD:SOT-23-6
- U3: value LIS3MDLTR -> QMC5883P; footprint Package_LGA:LGA-12_2x2mm_P0.5mm -> Package_LGA:LGA-16_3x3mm_P0.5mm
- moved C2 9.71 mm to (140.0, 157.5), turned to -90 degrees
- moved U1 5.05 mm to (143.0, 157.6), turned to -90 degrees
- moved C1 4.03 mm to (138.0, 157.5), turned to -90 degrees
- moved J1 1.00 mm to (151.5, 147.3)
- moved U3 0.56 mm to (147.8, 111.5)
- renumbered C9 to C10, C13 to C11, C7 to C12, C8 to C13, C10 to C14, C11 to C15, C16 to C18, C17 to C19, C18 to C20, C19 to C21, C12 to C22, C20 to C23, C21 to C24, C22 to C25, C24 to C26, C23 to C28, C26 to C29, C25 to C30, C3 to C6, C4 to C7, C5 to C8, C6 to C9, D5 to D1, D1 to D2, D2 to D3, D3 to D4, D4 to D5, J9 to J10, J10 to J11, J11 to J12, J12 to J13, J13 to J14, J17 to J15, J14 to J16, J16 to J17, J15 to J18, J25 to J19, J18 to J20, J19 to J21, J21 to J22, J22 to J23, J27 to J24, J20 to J25, J23 to J26, J24 to J27, J26 to J8, J8 to J9, R9 to R11, R10 to R12, R12 to R13, R13 to R14, R11 to R16, R14 to R17, R16 to R18, R17 to R20, R18 to R21, R3 to R4, R5 to R6, R7 to R9
Connections:
- C1 pad 1: +5V -> Net-(U1-SW)
- C1 pad 2: GND -> Net-(U1-BOOT)
- C2 pad 1: +3.3V -> +5V
- U1 pad 1: +5V -> GND
- U1 pad 2: GND -> Net-(U1-SW)
- U1 pad 3: +3.3V -> +5V
- U1 pad 4: GND -> Net-(U1-FB)
- U3 pad 10: +3.3V -> Net-(U3-C1)
- U3 pad 11: /I2C_SDA -> GND
- U3 pad 12: GND -> unconnected-(U3-NC-Pad12)
- U3 pad 2: GND -> +3.3V
- U3 pad 3: GND -> unconnected-(U3-NC-Pad3)
- U3 pad 4: Net-(U3-C1) -> unconnected-(U3-NC-Pad4)
- U3 pad 5: +3.3V -> unconnected-(U3-NC-Pad5)
- U3 pad 6: +3.3V -> unconnected-(U3-NC-Pad6)
Routing:
- net GND: track 71.0 -> 64.4 mm, vias 38 -> 34
- net +5V: track 4.72 -> 0.00 mm, vias 1 -> 0
- net +3.3V: track 78.9 -> 75.0 mm, vias 30 -> 27
- net /I2C_SDA: track 22.1 -> 23.3 mm
- net Net-(U3-C1): track 4.16 -> 5.35 mm

Commit message: changed the regulator to a buck converter
Routing:
- net +3.3V: track 75.0 -> 91.7 mm, vias 27 -> 28
- net Net-(U1-FB): track 0.00 -> 14.7 mm
- net Net-(U1-SW): track 0.00 -> 8.81 mm
- net Net-(U1-BOOT): track 0.00 -> 8.05 mm
- net GND: track 64.4 -> 71.3 mm, vias 34 -> 37
- net +5V: track 0.00 -> 3.12 mm, vias 0 -> 1
